File: kicad/ELH_02/ELH_02.kicad_sch (KiCad schematic)
At the start: 0 parts

Commit message: Attempt to commit changes
Parts:
- added BT1: Battery, symbol Device:Battery
- added C1, C13, C14, C15, C4: C_Small, symbol Device:C_Small
- added C10, C11, C12, C16, C2, C6, C7, C8, C9: C_Polarized, symbol Device:C_Polarized
- added C3, C5: C_Polarized_Small, symbol Device:C_Polarized_Small
- added U20: ~, symbol C_sym:MP1584
- added U9: LP5907MFX-3.3, Package_TO_SOT_SMD:SOT-23-5, symbol Regulator_Linear:LP5907MFX-3.3
Connections:
- new net: BT1.1 (+), C4.1, U20. (IN-)
- new net: BT1.2 (-), C4.2, U20. (IN-)
- new net GND_ESP32: C10.2, C11.2, C12.2, C13.1, C14.1, C15.2, C16.2, C5.2, C6.2, C7.2, C8.2, C9.2, U20. (IN-), U9.2 (GND)
- new net VCC_ESP32: C10.1, C11.1, C12.1, C13.2, C15.1, C16.1, C5.1, C6.1, C7.1, C8.1, C9.1, U20. (IN-), U9.1 (IN)
- new net VCC_SENS: C14.2, U9.5 (OUT)
- no-connect marks 0 -> 7
Other:
- added sheet gauges (gauges_file.kicad_sch)
- added sheet processing_and_data (processing_and_data_file.kicad_sch)
- added sheet sensing (sensing_file.kicad_sch)
- note added: "AIRFRAME-01 HX711 modules Power Supply Circuit"
- note added: "BUCK-01 HX711 modules Power Supply Circuit"
- note added: "Battery power circuit - Buck - LDO - ESP32 - SD - HX711 modules"
- note added: "Ceramic"
- note added: "ESP32 Power Supply Circuit"
- note added: "Electrolytic"
- note added: "MicroSD module Power Supply Circuit"
- note added: "Tantalum"
- title: (none) -> POWER SUBSYSTEM

Commit message: Preliminary solution to requested changes
Parts:
- removed C1: C_Small, symbol Device:C_Small
- removed C10, C11, C12, C2, C6, C7, C8, C9: C_Polarized, symbol Device:C_Polarized
- removed C3: C_Polarized_Small, symbol Device:C_Polarized_Small
- removed U9: LP5907MFX-3.3, Package_TO_SOT_SMD:SOT-23-5, symbol Regulator_Linear:LP5907MFX-3.3
- added ADT1, ADT2, ADT3, ADT7410: Sensor, symbol ELH_03_symbol:ADT7410
- added Ceramic_Capacitor: Capacitor, symbol Device:C_Small
- added ESP32_S3: Microcontroller, symbol C_sym:ESP32-S3-DevKitC-1
- added ICM20649: Sensor, symbol C_sym:ICM-20649
- added MAX4466: Microphone, symbol C_sym:MAX4466
- added MCP1700-3302E/TO: Regulator, symbol C_sym:MCP1700-3302E/TO
- added MPU6050 (x2): Sensor, symbol C_sym:MPU6050
- added MS5611: Sensor, symbol C_sym:MS5611
- added Micro_SD_Module: Micro SD Module, symbol C_sym:Micro_SD_Module
- added SS-12D00: Switch, symbol C_sym:Switch_3P_SS-12D00
- added W25Q128: Flash Card, symbol C_sym:W25Q128
- Ceramic_Capacitor: renamed from C14; value C_Small -> Capacitor
- Ceramic_Capacitor: renamed from C15; value C_Small -> Capacitor
- Ceramic_Capacitor: renamed from C4; value C_Small -> Capacitor
- Ceramic_Capacitor: renamed from C13; value C_Small -> Capacitor
- Electrolytic_Capacitor: renamed from C16; value C_Polarized -> Capacitor
- MP1584: renamed from U20; value ~ -> Regulator
- Tantalum_Capacitor: renamed from C5; value C_Polarized_Small -> Capacitor
- renumbered BT1 to 2S_Lithium-ion
Connections:
- net VCC_SENS is gone; now on net GND: Ceramic_Capacitor.2
- net GND_ESP32 renamed GND
- net GND: now also ADT1.2 (GND), ADT2.2 (GND), ADT3.2 (GND), ADT7410.2 (GND), Ceramic_Capacitor.2, ESP32_S3. (GND), ICM20649.3 (GND), MAX4466.2 (GND), MCP1700-3302E/TO.1 (GND), MPU6050.2 (GND), MPU6050.2 (GND), MS5611.2 (GND), Micro_SD_Module.6 (GND), SS-12D00.3 (GND), W25Q128.4 (GND); no longer Ceramic_Capacitor.1
- net VCC_ESP32 renamed +5V
- net +5V: now also Ceramic_Capacitor.1, ESP32_S3. (GND), MCP1700-3302E/TO.2 (VIN), W25Q128.1 (VCC); no longer Electrolytic_Capacitor.1
- new net: ESP32_S3. (GND), SS-12D00.2 (COM)
- new net +3V3: ADT1.1 (VIN), ADT2.1 (VIN), ADT3.1 (VIN), ADT7410.1 (VIN), Ceramic_Capacitor.1, Electrolytic_Capacitor.1, ICM20649.1 (VIN), MAX4466.3 (VCC), MCP1700-3302E/TO.3 (VOUT), MPU6050.1 (VCC), MPU6050.1 (VCC), MS5611.1 (VCC), Micro_SD_Module.1 (3V3), SS-12D00.1 (3V3)
- new net CS_ALT: ESP32_S3. (GND), MS5611.5 (CSB)
- new net CS_FLASH: ESP32_S3. (GND), W25Q128.2 (CS)
- new net CS_IMU: ESP32_S3. (GND), ICM20649.11 (CS)
- new net CS_SD: ESP32_S3. (GND), Micro_SD_Module.2 (CS)
- new net DT_AIRF011: ESP32_S3. (GND)
- new net DT_AIRF012: ESP32_S3. (GND)
- new net DT_AIRF013: ESP32_S3. (GND)
- new net DT_AIRF014: ESP32_S3. (GND)
- new net DT_BULK011: ESP32_S3. (GND)
- new net DT_BULK012: ESP32_S3. (GND)
- new net DT_BULK013: ESP32_S3. (GND)
- new net MIC: ESP32_S3. (GND), MAX4466.1 (OUT)
- new net MISO: ESP32_S3. (GND), Micro_SD_Module.5 (MISO), W25Q128.3 (DO)
- new net MOSI: ESP32_S3. (GND), Micro_SD_Module.3 (MOSI), W25Q128.6 (DI)
- new net SCK: ESP32_S3. (GND), Micro_SD_Module.4 (CLK), W25Q128.5 (CLK)
- new net SCK_AIRF011: ESP32_S3. (GND)
- new net SCK_AIRF012: ESP32_S3. (GND)
- new net SCK_AIRF013: ESP32_S3. (GND)
- new net SCK_AIRF014: ESP32_S3. (GND)
- new net SCK_BULK011: ESP32_S3. (GND)
- new net SCK_BULK012: ESP32_S3. (GND)
- new net SCK_BULK013: ESP32_S3. (GND)
- new net SCL: ADT1.3 (SCL), ADT2.3 (SCL), ADT3.3 (SCL), ADT7410.3 (SCL), ESP32_S3. (GND), ICM20649.4 (SCL), MPU6050.3 (SCL), MPU6050.3 (SCL), MS5611.3 (SCL)
- new net SDA: ADT1.4 (SDA), ADT2.4 (SDA), ADT3.4 (SDA), ADT7410.4 (SDA), ESP32_S3. (GND), ICM20649.5 (SDA), MPU6050.4 (SDA), MPU6050.4 (SDA), MS5611.4 (SDA)
- no-connect marks 7 -> 34
Other:
- removed sheet processing_and_data
- removed sheet sensing
- note added: "3,3V Output"
- note added: "5V Input"
- note added: "5V Output"
- note added: "7,4V Input"
- note added: "ADT-7410"
- note added: "Battery power circuit - Buck - LDO"
- note added: "DATA STORAGE CIRCUIT"
- note added: "ICM-20649"
- note added: "MAX4466"
- note added: "MPU-6050"
- note added: "MS5611"
- note added: "PROCESSING CIRCUIT"
- note removed: "AIRFRAME-01 HX711 modules Power Supply Circuit"
- note removed: "BUCK-01 HX711 modules Power Supply Circuit"
- note removed: "Battery power circuit - Buck - LDO - ESP32 - SD - HX711 modules"
- note removed: "Ceramic"
- note removed: "ESP32 Power Supply Circuit"
- note removed: "Electrolytic"
- note removed: "MicroSD module Power Supply Circuit"
- note removed: "Tantalum"
- moved on the sheet: 2S_Lithium-ion
